File: KiCAD Files/PCB_Christmas_Tree/PCB_Christmas_Tree.kicad_pcb (KiCad board)
At the start: 2 copper layers, 127 x 60 mm, 69 parts, among them J1 Conn_01x03_Pin, J2 CR2032, J3 Conn_01x05_Pin, J4 Conn_01x05_Pin, J5 Conn_01x05_Pin, J6 Conn_01x05_Pin, Q1 PMOS, Q2 PMOS, Q3 PMOS, Q4 NPN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

Commit message: schematic revision
Parts:
- removed J6: Conn_01x05_Pin, LocalFootprintLib:Multi_board_connector
- removed Q6: PMOS, Package_TO_SOT_SMD:SOT-323_SC-70_Handsoldering
- removed R6: 1k, Resistor_SMD:R_0603_1608Metric_Pad0.98x0.95mm_HandSolder
- added J7: Conn_01x04_Pin, LocalFootprintLib:Multi_board_connector, F.Cu at (81.3, 101.0)
- D11, D13, D15, D17, D19, D20, D24, D25, D6, D7, D8, D9, R11, R12, R13, R14, R16, R18, R20, R22, R24, R25, R29, R30: moved to B.Cu
- J3, J4, J5: value Conn_01x05_Pin -> Conn_01x04_Pin
- moved D24 298.2 mm to (176.0, 103.8), turned to 180 degrees
- moved R29 289.5 mm to (171.4, 102.5), turned to 180 degrees
- moved R16 273.2 mm to (181.4, 125.6), turned to 0 degrees
- moved D16 266.5 mm to (172.5, 120.2)
- moved R21 266.5 mm to (176.2, 120.4)
- moved D11 265.4 mm to (177.4, 125.6), turned to 180 degrees
- moved D2 260.9 mm to (168.0, 97.9)
- moved R7 260.9 mm to (171.8, 97.9)
- moved D17 229.5 mm to (129.4, 123.4), turned to 0 degrees
- moved R22 223.0 mm to (125.4, 123.3), turned to 180 degrees
- moved D8 221.1 mm to (109.7, 127.3), turned to 0 degrees
- moved D25 214.8 mm to (95.2, 85.6)
- moved R13 214.5 mm to (105.7, 127.3), turned to 180 degrees
- moved D15 211.5 mm to (161.2, 73.0), turned to 0 degrees
- moved D4 211.4 mm to (159.3, 76.0)
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Connections:
- D11 pad 2: /LED_Power_4 -> /LED_Power_1
- D13 pad 2: /LED_Power_4 -> /LED_Power_1
- D15 pad 2: /LED_Power_4 -> /LED_Power_2
- D17 pad 2: /LED_Power_4 -> /LED_Power_2
- D20 pad 2: /LED_Power_4 -> /LED_Power_3
- D24 pad 2: /LED_Power_4 -> /LED_Power_3
- J1 pad 2: /Switch_in -> /UDPI
- J3 pad 4: /LED_Power_4 -> GND
- J4 pad 4: /LED_Power_4 -> GND
- J5 pad 4: /LED_Power_4 -> GND
- U1 pad 3: /LED_Set_4 -> /LED_Set_3
- U1 pad 6: /Switch_in -> /UDPI
Routing:
- net VDD: track 48.7 -> 0.00 mm
- net +BATT: track 33.5 -> 0.00 mm
- net Net-(D1-K): track 14.8 -> 0.00 mm, vias 1 -> 0
- net /Switch_in: track 14.1 -> 0.00 mm, vias 1 -> 0
- net Net-(Q1-G): track 10.6 -> 0.00 mm
- net /LED_Set_4: track 8.31 -> 0.00 mm
- net /LED_Set_3: track 7.25 -> 0.00 mm
- net /LED_Set_2: track 6.95 -> 0.00 mm
- net /LED_Set_1: track 4.83 -> 0.00 mm
- net /Power_sustain: track 4.65 -> 0.00 mm
- net Net-(Q4-B): track 3.08 -> 0.00 mm
- net Net-(Q3-G): track 2.81 -> 0.00 mm
- net Net-(Q5-G): track 2.78 -> 0.00 mm
- net Net-(Q6-G): track 2.73 -> 0.00 mm
- net Net-(Q2-G): track 2.63 -> 0.00 mm
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Other:
- board size 127 x 60 mm -> 129.4 x 60.1 mm

Commit message: pcb revision
Parts:
- moved D11 72.1 mm to (248.0, 140.0), turned to 0 degrees
- moved R16 63.2 mm to (243.0, 140.0), turned to 180 degrees
- moved D15 61.9 mm to (223.1, 76.0)
- moved R20 61.9 mm to (219.0, 76.0)
- moved D24 61.1 mm to (237.0, 106.0), turned to 0 degrees
- moved R29 60.7 mm to (232.0, 106.0)
- moved R18 55.5 mm to (185.0, 92.0)
- moved D16 55.5 mm to (228.0, 120.0), turned to 90 degrees
- moved R25 54.7 mm to (196.0, 58.0)
- moved D20 54.3 mm to (198.0, 54.0), turned to 90 degrees
- moved R21 53.9 mm to (230.0, 124.0)
- moved D13 53.8 mm to (187.0, 88.0), turned to 90 degrees
- moved D4 53.4 mm to (208.0, 54.0), turned to 90 degrees
- moved D2 52.9 mm to (220.0, 88.0), turned to 90 degrees
- moved R22 50.7 mm to (176.1, 125.0)
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Connections:
- U1 pad 3: /LED_Set_3 -> /Switch_in
Routing:
- net /LED_Power_3: track 0.00 -> 395.9 mm, vias 0 -> 9
- net /LED_Power_2: track 0.00 -> 346.2 mm, vias 0 -> 9
- net /LED_Power_1: track 0.00 -> 346.0 mm, vias 0 -> 10
- net VDD: track 0.00 -> 46.5 mm
- net +BATT: track 0.00 -> 34.0 mm
- net /UDPI: track 0.00 -> 21.2 mm, vias 0 -> 1
- net Net-(Q1-G): track 0.00 -> 10.6 mm
- net Net-(D1-K): track 0.00 -> 9.27 mm, vias 0 -> 1
- net /LED_Set_3: track 0.00 -> 8.77 mm
- net /LED_Set_2: track 0.00 -> 6.80 mm
- net /Switch_in: track 0.00 -> 6.24 mm
- net Net-(D18-K): track 0.00 -> 4.84 mm
- net Net-(D17-K): track 0.00 -> 4.83 mm
- net /LED_Set_1: track 0.00 -> 4.83 mm
- net /Power_sustain: track 0.00 -> 4.66 mm
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- added copper zone on B.Cu, net GND
- added copper zone on F.Cu, net GND
Other:
- board size 129.4 x 60.1 mm -> 207.1 x 98.8 mm

Commit message: pcb update
Parts:
- moved D25 5.17 mm to (112.3, 73.9)
- moved R30 5.01 mm to (108.4, 73.9)
- moved R20 4.09 mm to (215.6, 73.7)
- moved D15 4.09 mm to (219.7, 73.7)
- moved D10 4.08 mm to (79.5, 73.9)
- moved D11 3.98 mm to (244.3, 138.4)
- moved R16 3.98 mm to (239.3, 138.4)
- moved D23 3.54 mm to (65.0, 104.1)
- moved D5 3.42 mm to (162.6, 137.9)
- moved R10 3.42 mm to (166.6, 137.9)
- moved R28 3.30 mm to (68.8, 104.1)
- moved D3 3.24 mm to (171.9, 104.6)
- moved R8 3.24 mm to (176.0, 104.6)
- moved R15 3.11 mm to (83.3, 73.9)
- moved D24 3.02 mm to (234.2, 104.9)
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Routing:
- net /LED_Power_2: track 346.2 -> 327.7 mm
- net /LED_Power_1: track 346.0 -> 360.9 mm, vias 10 -> 6
- net /LED_Power_3: track 395.9 -> 386.3 mm, vias 9 -> 10
- net Net-(D1-K): track 9.27 -> 17.2 mm
- net Net-(D10-K): track 3.06 -> 1.87 mm
- net Net-(D19-K): track 3.06 -> 2.13 mm
- net Net-(D22-K): track 3.00 -> 2.38 mm
- net GND: vias 42 -> 50
Other:
- outline, holes or cut-outs redrawn

Commit message: schematic update, footprint revision
Parts:
- removed R3: 1k, Resistor_SMD:R_0603_1608Metric_Pad0.98x0.95mm_HandSolder
- added Rq1: 10k, Resistor_SMD:R_0603_1608Metric_Pad0.98x0.95mm_HandSolder, B.Cu at (83.0, 158.6)
- Q1, Q2, Q3, Q5: value PMOS -> AO3401A; footprint Package_TO_SOT_SMD:SOT-323_SC-70_Handsoldering -> Package_TO_SOT_SMD:SOT-23
- Q4: value NPN -> BC817
- R1: value 100k -> 10k
- R2, R5: value 1k -> 10k
- moved Q5 47.9 mm to (87.7, 171.7), turned to 180 degrees
- moved Q3 38.3 mm to (87.7, 162.8), turned to 180 degrees
- moved Q4 32.1 mm to (87.7, 167.3)
- moved R5 31.4 mm to (83.0, 156.0)
- moved Q2 28.9 mm to (87.7, 158.4), turned to 180 degrees
- moved Q1 26.3 mm to (87.7, 153.9)
- moved R2 23.1 mm to (83.0, 151.0)
- moved R1 19.4 mm to (83.0, 148.5), turned to 180 degrees
- moved R4 18.6 mm to (83.0, 153.5), turned to 180 degrees
- moved D1 12.0 mm to (90.7, 145.8)
- moved U1 1.70 mm to (95.5, 137.4), turned to 180 degrees
Connections:
- Q1 pad 1: VDD -> Net-(Q1-G)
- Q1 pad 2: Net-(Q1-G) -> +BATT
- Q1 pad 3: +BATT -> VDD
- Q2 pad 1: /LED_Power_3 -> Net-(Q2-G)
- Q2 pad 2: Net-(Q2-G) -> VDD
- Q2 pad 3: VDD -> /LED_Power_3
- Q3 pad 1: /LED_Power_1 -> Net-(Q3-G)
- Q3 pad 2: Net-(Q3-G) -> VDD
- Q3 pad 3: VDD -> /LED_Power_1
- Q4 pad 1: Net-(Q1-G) -> Net-(Q4-B)
- Q4 pad 2: Net-(Q4-B) -> GND
- Q4 pad 3: GND -> Net-(Q1-G)
- Q5 pad 1: /LED_Power_2 -> Net-(Q5-G)
- Q5 pad 2: Net-(Q5-G) -> VDD
- Q5 pad 3: VDD -> /LED_Power_2
- U1 pad 2: /LED_Set_3 -> /Power_sustain
- U1 pad 4: /Power_sustain -> /LED_Set_3
Routing:
- net VDD: track 46.5 -> 0.00 mm
- net +BATT: track 34.0 -> 0.00 mm
- net /LED_Power_3: track 386.3 -> 361.7 mm, vias 10 -> 9
- net /UDPI: track 21.2 -> 0.00 mm, vias 1 -> 0
- net Net-(Q1-G): track 10.6 -> 0.00 mm
- net Net-(D1-K): track 17.2 -> 7.95 mm, vias 1 -> 0
- net /LED_Set_3: track 8.77 -> 0.00 mm
- net /LED_Power_1: track 360.9 -> 352.2 mm, vias 6 -> 5
- net /LED_Power_2: track 327.7 -> 319.7 mm, vias 9 -> 8
- net /LED_Set_2: track 6.80 -> 0.00 mm
- net /Switch_in: track 6.24 -> 0.00 mm
- net /LED_Set_1: track 4.83 -> 0.00 mm
- net /Power_sustain: track 4.66 -> 0.00 mm
- net Net-(Q4-B): track 3.17 -> 0.00 mm
- net Net-(Q3-G): track 2.81 -> 0.00 mm
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
Commit message: pcb updates
Parts:
- moved Q5 44.5 mm to (102.7, 129.9), turned to 90 degrees
- moved Q3 35.2 mm to (98.3, 129.3), turned to 90 degrees
- moved Rq1 29.9 mm to (99.2, 133.3), turned to 0 degrees
- moved Q2 29.7 mm to (94.0, 129.4), turned to 90 degrees
- moved Q4 29.2 mm to (83.4, 138.4)
- moved R5 27.2 mm to (102.6, 137.2), turned to 90 degrees
- moved Q1 22.5 mm to (90.2, 131.6), turned to 90 degrees
- moved R2 21.1 mm to (94.5, 133.3), turned to 0 degrees
- moved R4 15.4 mm to (88.6, 139.2), turned to 0 degrees
- moved R1 14.2 mm to (82.8, 134.4), turned to -90 degrees
- moved D1 9.83 mm to (88.6, 136.1)
- moved U1 0.80 mm to (96.2, 137.6), turned to 0 degrees
Routing:
- net VDD: track 0.00 -> 64.3 mm
- net +BATT: track 0.00 -> 34.1 mm
- net /LED_Power_2: track 319.7 -> 348.9 mm, vias 8 -> 7
- net /UDPI: track 0.00 -> 15.1 mm
- net Net-(Q1-G): track 0.00 -> 13.8 mm
- net Net-(D1-K): track 7.95 -> 15.8 mm, vias 0 -> 1
- net /LED_Power_1: track 352.2 -> 359.1 mm, vias 5 -> 6
- net Net-(Q5-G): track 0.00 -> 5.86 mm
- net /Power_sustain: track 0.00 -> 4.59 mm
- net /LED_Power_3: track 361.7 -> 366.3 mm, vias 9 -> 10
- net /Switch_in: track 0.00 -> 4.22 mm
- net Net-(Q4-B): track 0.00 -> 4.14 mm
- net /LED_Set_2: track 0.00 -> 3.98 mm
- net Net-(Q3-G): track 0.00 -> 3.45 mm
- net Net-(Q2-G): track 0.00 -> 3.22 mm
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
Commit message: pcb modifications
Parts:
- added REF**: SolderWirePad_1x01_SMD_1x2mm, Connector_Wire:SolderWirePad_1x01_SMD_1x2mm, F.Cu at (94.5, 48.6)
- added REF**: SolderWirePad_1x01_SMD_1x2mm, Connector_Wire:SolderWirePad_1x01_SMD_1x2mm, F.Cu at (204.5, 49.1)
- added REF**: SolderWirePad_1x01_SMD_1x2mm, Connector_Wire:SolderWirePad_1x01_SMD_1x2mm, F.Cu at (201.5, 49.1)
- added REF**: SolderWirePad_1x01_SMD_1x2mm, Connector_Wire:SolderWirePad_1x01_SMD_1x2mm, F.Cu at (97.4, 48.6)
- added REF**: SolderWirePad_1x01_SMD_1x2mm, Connector_Wire:SolderWirePad_1x01_SMD_1x2mm, B.Cu at (201.5, 49.1)
- added REF**: SolderWirePad_1x01_SMD_1x2mm, Connector_Wire:SolderWirePad_1x01_SMD_1x2mm, B.Cu at (204.5, 49.1)
- added REF**: SolderWirePad_1x01_SMD_1x2mm, Connector_Wire:SolderWirePad_1x01_SMD_1x2mm, B.Cu at (97.4, 48.6)
- added REF**: SolderWirePad_1x01_SMD_1x2mm, Connector_Wire:SolderWirePad_1x01_SMD_1x2mm, B.Cu at (94.5, 48.6)
Routing:
- net /LED_Power_3: track 366.3 -> 356.2 mm, vias 10 -> 26
- net /LED_Power_1: track 359.1 -> 354.1 mm, vias 6 -> 22
- net /LED_Power_2: track 348.9 -> 344.6 mm, vias 7 -> 23
- net GND: vias 47 -> 63
Other:
- outline, holes or cut-outs redrawn
