File: KiCAD Files/Manufacturing_main/PCB_Christmas_Tree.kicad_pcb (KiCad board)
At the start: 2 copper layers, 100 x 98.6 mm, 41 parts, among them J1 Conn_01x03_Pin, J2 CR2032, J5 Conn_01x04_Pin, J7 Conn_01x04_Pin, Q1 PMOS, Q2 PMOS, Q3 PMOS, Q4 NPN, Q5 PMOS, SW1 SW_Omron_B3FS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

Commit message: v2 added
Parts:
- removed D18, D19, D21, D23, D25, D6, D7, D8, D9: LED, LED_SMD:LED_0805_2012Metric_Pad1.15x1.40mm_HandSolder
- removed J5, J7: Conn_01x04_Pin, LocalFootprintLib:Multi_board_connector
- removed R11, R12, R13, R23, R24, R27, R30: 100, Resistor_SMD:R_0603_1608Metric_Pad0.98x0.95mm_HandSolder
- added D11: LED, LED_SMD:LED_0805_2012Metric_Pad1.15x1.40mm_HandSolder, B.Cu at (106.1, 47.5)
- added D13: LED, LED_SMD:LED_0805_2012Metric_Pad1.15x1.40mm_HandSolder, B.Cu at (86.1, 114.5)
- added D14: LED, LED_SMD:LED_0805_2012Metric_Pad1.15x1.40mm_HandSolder, F.Cu at (93.6, 68.4)
- added D16: LED, LED_SMD:LED_0805_2012Metric_Pad1.15x1.40mm_HandSolder, F.Cu at (114.1, 47.5)
- added D2: LED, LED_SMD:LED_0805_2012Metric_Pad1.15x1.40mm_HandSolder, F.Cu at (79.1, 98.6)
- added D24: LED, LED_SMD:LED_0805_2012Metric_Pad1.15x1.40mm_HandSolder, B.Cu at (126.4, 68.4)
- added D3: LED, LED_SMD:LED_0805_2012Metric_Pad1.15x1.40mm_HandSolder, F.Cu at (67.4, 132.9)
- added D4: LED, LED_SMD:LED_0805_2012Metric_Pad1.15x1.40mm_HandSolder, F.Cu at (127.1, 83.5)
- added D5: LED, LED_SMD:LED_0805_2012Metric_Pad1.15x1.40mm_HandSolder, F.Cu at (134.1, 113.5)
- added J3: Conn_01x04_Pin, LocalFootprintLib:Multi_board_connector, F.Cu at (107.8, 95.1)
- added J6: Conn_01x04_Pin, LocalFootprintLib:Multi_board_connector, B.Cu at (112.2, 95.1)
- added R16: 100, Resistor_SMD:R_0603_1608Metric_Pad0.98x0.95mm_HandSolder, B.Cu at (147.7, 132.7)
- added R18: 100, Resistor_SMD:R_0603_1608Metric_Pad0.98x0.95mm_HandSolder, F.Cu at (97.4, 68.4)
- added R20: 100, Resistor_SMD:R_0603_1608Metric_Pad0.98x0.95mm_HandSolder, F.Cu at (116.1, 52.5)
- added R6: 100, Resistor_SMD:R_0603_1608Metric_Pad0.98x0.95mm_HandSolder, F.Cu at (82.9, 98.6)
- added R7: 100, Resistor_SMD:R_0603_1608Metric_Pad0.98x0.95mm_HandSolder, F.Cu at (71.8, 132.9)
- added R8: 100, Resistor_SMD:R_0603_1608Metric_Pad0.98x0.95mm_HandSolder, F.Cu at (129.0, 88.5)
- added R9: 100, Resistor_SMD:R_0603_1608Metric_Pad0.98x0.95mm_HandSolder, F.Cu at (137.1, 118.5)
- added REF**: SolderWirePad_1x01_SMD_1x2mm, Connector_Wire:SolderWirePad_1x01_SMD_1x2mm, F.Cu at (111.5, 43.1)
- added REF**: SolderWirePad_1x01_SMD_1x2mm, Connector_Wire:SolderWirePad_1x01_SMD_1x2mm, F.Cu at (108.6, 43.1)
- added REF**: SolderWirePad_1x01_SMD_1x2mm, Connector_Wire:SolderWirePad_1x01_SMD_1x2mm, B.Cu at (108.6, 43.1)
- added REF**: SolderWirePad_1x01_SMD_1x2mm, Connector_Wire:SolderWirePad_1x01_SMD_1x2mm, B.Cu at (111.5, 43.1)
- D10, D12, D22, R15, R17, R26, R28: moved to B.Cu
- J1: value Conn_01x03_Pin -> CR2032; footprint Connector_PinHeader_2.54mm:PinHeader_1x03_P2.54mm_Vertical -> LocalFootprintLib:BC-2002; moved to F.Cu
- J2: value CR2032 -> Conn_01x03_Pin; footprint LocalFootprintLib:BC-2002 -> Connector_PinHeader_2.54mm:PinHeader_1x03_P2.54mm_Vertical; moved to B.Cu
- Q1, Q2, Q3, Q5: value PMOS -> AO3401A
- Q4: value NPN -> BC817
- R1: value 100k -> 10k
- R2, R3, R5: value 1k -> 10k
- moved D22 97.0 mm to (141.9, 98.6), turned to 0 degrees
- moved D12 95.0 mm to (151.8, 132.7), turned to 0 degrees
- moved R28 64.5 mm to (122.5, 68.4), turned to 180 degrees
- moved R17 64.1 mm to (84.1, 119.5), turned to 180 degrees
- moved R14 42.7 mm to (92.1, 88.5)
- moved J2 33.6 mm to (129.6, 133.5), turned to 90 degrees
- moved R15 29.8 mm to (104.1, 52.5), turned to 180 degrees
- moved R26 23.3 mm to (137.8, 98.6), turned to 180 degrees
- moved Q1 18.6 mm to (108.1, 123.9), turned to 90 degrees
- moved R1 17.9 mm to (108.6, 127.8)
- moved D10 17.5 mm to (94.1, 83.5), turned to 90 degrees
- moved R5 17.4 mm to (116.7, 131.5), turned to 90 degrees
- moved Q5 17.3 mm to (116.8, 124.4)
- moved SW1 15.1 mm to (91.1, 130.3)
- moved U1 15.0 mm to (110.3, 132.1), turned to 0 degrees
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Connections:
- D1 pad 1: Net-(Q1-G) -> Net-(Q3-G)
- D10 pad 2: /LED_Power_2 -> /LED_Power_1
- D12 pad 2: /LED_Power_2 -> /LED_Power_1
- D22 pad 2: /LED_Power_1 -> /LED_Power_2
- J1 pad 1: VDD -> +BATT
- J1 pad 2: /UDPI -> GND
- J2 pad 1: +BATT -> VDD
- J2 pad 2: GND -> /UDPI
- Q1 pad 1: VDD -> Net-(Q1-G)
- Q1 pad 2: Net-(Q1-G) -> VDD
- Q1 pad 3: +BATT -> /LED_Power_3
- Q2 pad 1: /LED_Power_3 -> Net-(Q2-G)
- Q2 pad 2: Net-(Q2-G) -> VDD
- Q2 pad 3: VDD -> /LED_Power_1
- Q3 pad 1: /LED_Power_1 -> Net-(Q3-G)
- Q3 pad 2: Net-(Q3-G) -> +BATT
- Q4 pad 1: Net-(Q1-G) -> Net-(Q4-B)
- Q4 pad 2: Net-(Q4-B) -> GND
- Q4 pad 3: GND -> Net-(Q3-G)
- Q5 pad 1: /LED_Power_2 -> Net-(Q5-G)
- Q5 pad 2: Net-(Q5-G) -> VDD
- Q5 pad 3: VDD -> /LED_Power_2
- R1 pad 1: +BATT -> /LED_Set_3
- R14 pad 1: Net-(D9-K) -> Net-(D10-K)
- R15 pad 1: Net-(D10-K) -> (no net)
- R17 pad 1: Net-(D12-K) -> (no net)
- R2 pad 1: /LED_Set_3 -> /LED_Set_1
- R26 pad 1: Net-(D21-K) -> Net-(D22-K)
- R28 pad 1: Net-(D23-K) -> (no net)
- R3 pad 1: /LED_Set_1 -> +BATT
- U1 pad 2: /LED_Set_3 -> /Power_sustain
- U1 pad 4: /Power_sustain -> /LED_Set_3
Routing:
- net (no net): track 0.00 -> 31.1 mm
- net /LED_Power_3: track 201.9 -> 177.8 mm, vias 6 -> 12
- net /LED_Power_2: track 193.1 -> 215.6 mm, vias 6 -> 12
- net VDD: track 46.5 -> 66.8 mm
- net Net-(Q3-G): track 2.81 -> 13.6 mm
- net Net-(Q1-G): track 10.6 -> 2.95 mm
- net /LED_Set_3: track 8.77 -> 2.46 mm
- net /LED_Power_1: track 205.0 -> 211.2 mm, vias 5 -> 13
- net /UDPI: track 21.2 -> 15.1 mm, vias 1 -> 0
- net Net-(D18-K): track 4.84 -> 0.00 mm
- net Net-(D7-K): track 4.45 -> 0.00 mm
- net Net-(D9-K): track 4.43 -> 0.00 mm
- net Net-(D6-K): track 4.43 -> 0.00 mm
- net Net-(D21-K): track 4.39 -> 0.00 mm
- net /LED_Set_2: track 6.80 -> 4.05 mm
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Other:
- board text added: "GND"
- board text added: "J4"
- board text added: "UPDI"
- board text added: "VDD"

Commit message: Dodano pliki gerber v1
Parts:
- removed the REF** at (111.5, 43.1) (x2)
- removed the REF** at (108.6, 43.1) (x2)
- added REF**: SolderWirePad_1x01_SMD_1x2mm, Connector_Wire:SolderWirePad_1x01_SMD_1x2mm, F.Cu at (151.0, 44.2)
- added REF**: SolderWirePad_1x01_SMD_1x2mm, Connector_Wire:SolderWirePad_1x01_SMD_1x2mm, F.Cu at (148.1, 44.2)
- added REF**: SolderWirePad_1x01_SMD_1x2mm, Connector_Wire:SolderWirePad_1x01_SMD_1x2mm, B.Cu at (151.0, 44.2)
- added REF**: SolderWirePad_1x01_SMD_1x2mm, Connector_Wire:SolderWirePad_1x01_SMD_1x2mm, B.Cu at (148.1, 44.2)
- R1, R14, R15, R16, R17, R18, R2, R20, R26, R28, R3, R4, R5, R6, R7, R8, R9: footprint Resistor_SMD:R_0603_1608Metric_Pad0.98x0.95mm_HandSolder -> Resistor_SMD:R_0805_2012Metric_Pad1.20x1.40mm_HandSolder
- moved D1 39.6 mm to (142.3, 131.7)
- moved D14 39.6 mm to (133.1, 69.5)
- moved J6 39.6 mm to (151.8, 96.2)
- moved Q2 39.6 mm to (152.0, 124.9)
- moved Q3 39.6 mm to (143.8, 127.2)
- moved Q5 39.6 mm to (156.3, 125.5)
- moved R18 39.6 mm to (136.9, 69.5)
- moved R28 39.6 mm to (162.1, 69.5)
- moved R4 39.6 mm to (142.3, 134.8)
- moved R5 39.6 mm to (156.2, 132.6)
- moved SW1 39.6 mm to (130.6, 131.4)
- moved D10 39.6 mm to (133.6, 84.6)
- moved D11 39.6 mm to (145.6, 48.6)
- moved D12 39.6 mm to (191.3, 133.8)
- moved D13 39.6 mm to (125.6, 115.6)
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Connections:
- J2 pad 2: /UDPI -> GND
- J2 pad 3: GND -> /UDPI
Routing:
- net /UDPI: track 15.1 -> 12.6 mm
- net (no net): vias 0 -> 2
Other:
- board text added: "JLCJLCJLCJLC"
- board text removed: "J4"

Commit message: dodano gerbery bez napisu JLCJLCJLC
Other:
- board text removed: "JLCJLCJLCJLC"
