File: KiCAD Files/Manufacturing_slave/PCB_Christmas_Tree.kicad_pcb (KiCad board)
At the start: 2 copper layers, 100 x 98.6 mm, 26 parts, among them J3 Conn_01x04_Pin, J4 Conn_01x04_Pin

Commit message: v2 added
Parts:
- removed D11, D13, D14, D16, D2, D24, D3, D4, D5: LED, LED_SMD:LED_0805_2012Metric_Pad1.15x1.40mm_HandSolder
- removed J3: Conn_01x04_Pin, LocalFootprintLib:Multi_board_connector
- removed R16, R18, R20, R7, R8, R9: 100, Resistor_SMD:R_0603_1608Metric_Pad0.98x0.95mm_HandSolder
- added D18: LED, LED_SMD:LED_0805_2012Metric_Pad1.15x1.40mm_HandSolder, F.Cu at (181.6, 73.4)
- added D19: LED, LED_SMD:LED_0805_2012Metric_Pad1.15x1.40mm_HandSolder, B.Cu at (215.9, 73.4)
- added D21: LED, LED_SMD:LED_0805_2012Metric_Pad1.15x1.40mm_HandSolder, B.Cu at (175.2, 119.8)
- added D23: LED, LED_SMD:LED_0805_2012Metric_Pad1.15x1.40mm_HandSolder, B.Cu at (194.2, 53.8)
- added D25: LED, LED_SMD:LED_0805_2012Metric_Pad1.15x1.40mm_HandSolder, B.Cu at (230.4, 104.7)
- added D6: LED, LED_SMD:LED_0805_2012Metric_Pad1.15x1.40mm_HandSolder, F.Cu at (216.2, 87.8)
- added D7: LED, LED_SMD:LED_0805_2012Metric_Pad1.15x1.40mm_HandSolder, F.Cu at (168.1, 104.4)
- added D8: LED, LED_SMD:LED_0805_2012Metric_Pad1.15x1.40mm_HandSolder, F.Cu at (204.2, 53.8)
- added D9: LED, LED_SMD:LED_0805_2012Metric_Pad1.15x1.40mm_HandSolder, F.Cu at (158.8, 137.7)
- added J5: Conn_01x04_Pin, LocalFootprintLib:Multi_board_connector, B.Cu at (196.9, 100.5)
- added R11: 100, Resistor_SMD:R_0603_1608Metric_Pad0.98x0.95mm_HandSolder, F.Cu at (172.2, 104.4)
- added R12: 100, Resistor_SMD:R_0603_1608Metric_Pad0.98x0.95mm_HandSolder, F.Cu at (206.2, 57.8)
- added R13: 100, Resistor_SMD:R_0603_1608Metric_Pad0.98x0.95mm_HandSolder, F.Cu at (162.8, 137.7)
- added R23: 100, Resistor_SMD:R_0603_1608Metric_Pad0.98x0.95mm_HandSolder, B.Cu at (211.8, 73.4)
- added R24: 100, Resistor_SMD:R_0603_1608Metric_Pad0.98x0.95mm_HandSolder, F.Cu at (226.2, 123.8)
- added R27: 100, Resistor_SMD:R_0603_1608Metric_Pad0.98x0.95mm_HandSolder, B.Cu at (192.2, 57.8)
- added REF**: SolderWirePad_1x01_SMD_1x2mm, Connector_Wire:SolderWirePad_1x01_SMD_1x2mm, F.Cu at (200.7, 48.9)
- added REF**: SolderWirePad_1x01_SMD_1x2mm, Connector_Wire:SolderWirePad_1x01_SMD_1x2mm, F.Cu at (197.7, 48.9)
- added REF**: SolderWirePad_1x01_SMD_1x2mm, Connector_Wire:SolderWirePad_1x01_SMD_1x2mm, B.Cu at (197.7, 48.9)
- added REF**: SolderWirePad_1x01_SMD_1x2mm, Connector_Wire:SolderWirePad_1x01_SMD_1x2mm, B.Cu at (200.7, 48.9)
- D20, R22: moved to F.Cu
- R19, R21: moved to B.Cu
- moved R19 79.3 mm to (235.5, 138.2), turned to 180 degrees
- moved R25 70.9 mm to (172.3, 124.8)
- moved D20 70.8 mm to (224.2, 119.8)
- moved R10 69.2 mm to (218.2, 91.8)
- moved D15 67.8 mm to (240.5, 138.2)
- moved R21 58.5 mm to (181.2, 91.8), turned to 180 degrees
- moved R22 52.4 mm to (185.7, 73.4), turned to 0 degrees
- moved D17 32.5 mm to (183.2, 87.8)
- moved R29 3.82 mm to (225.4, 104.7)
- moved J4 3.82 mm to (201.4, 100.5)
Connections:
- D15 pad 2: /LED_Power_2 -> /LED_Power_1
- D17 pad 2: /LED_Power_2 -> /LED_Power_1
- D20 pad 2: /LED_Power_3 -> /LED_Power_2
- R10 pad 1: Net-(D5-K) -> (no net)
- R19 pad 1: Net-(D14-K) -> Net-(D15-K)
- R21 pad 1: Net-(D16-K) -> Net-(D17-K)
- R22 pad 1: Net-(D17-K) -> (no net)
- R25 pad 1: Net-(D20-K) -> (no net)
- R29 pad 1: Net-(D24-K) -> (no net)
Routing:
- net (no net): track 0.00 -> 26.7 mm
- net /LED_Power_3: track 184.5 -> 171.7 mm, vias 4 -> 12
- net /LED_Power_1: track 155.9 -> 146.4 mm, vias 1 -> 9
- net /LED_Power_2: track 134.7 -> 129.1 mm, vias 3 -> 10
- net Net-(D4-K): track 3.43 -> 0.00 mm
- net Net-(D2-K): track 3.43 -> 0.00 mm
- net Net-(D16-K): track 3.40 -> 0.00 mm
- net Net-(D13-K): track 3.40 -> 0.00 mm
- net Net-(D24-K): track 3.06 -> 0.00 mm
- net Net-(D11-K): track 3.06 -> 0.00 mm
- net Net-(D14-K): track 2.14 -> 0.00 mm
- net Net-(D3-K): track 2.13 -> 0.00 mm
- net Net-(D5-K): track 2.13 -> 0.00 mm
- net Net-(D17-K): track 4.83 -> 3.40 mm
- net Net-(D15-K): track 2.13 -> 3.06 mm
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Other:
- outline, holes or cut-outs redrawn

Commit message: Dodano pliki gerber v1
Parts:
- removed the REF** at (200.7, 48.9) (x2)
- removed the REF** at (197.7, 48.9) (x2)
- added G***: LOGO, LOGO, F.Cu at (83.8, 130.1)
- added G***: LOGO, LOGO, B.Cu at (81.8, 134.1)
- added REF**: SolderWirePad_1x01_SMD_1x2mm, Connector_Wire:SolderWirePad_1x01_SMD_1x2mm, F.Cu at (95.4, 49.2)
- added REF**: SolderWirePad_1x01_SMD_1x2mm, Connector_Wire:SolderWirePad_1x01_SMD_1x2mm, F.Cu at (98.3, 49.2)
- added REF**: SolderWirePad_1x01_SMD_1x2mm, Connector_Wire:SolderWirePad_1x01_SMD_1x2mm, B.Cu at (98.3, 49.2)
- added REF**: SolderWirePad_1x01_SMD_1x2mm, Connector_Wire:SolderWirePad_1x01_SMD_1x2mm, B.Cu at (95.4, 49.2)
- R10, R11, R12, R13, R19, R21, R22, R23, R24, R25, R27, R29: footprint Resistor_SMD:R_0603_1608Metric_Pad0.98x0.95mm_HandSolder -> Resistor_SMD:R_0805_2012Metric_Pad1.20x1.40mm_HandSolder
- moved D15 102.4 mm to (138.2, 138.5)
- moved D25 102.4 mm to (128.0, 105.0)
- moved J4 102.4 mm to (99.1, 100.8)
- moved R19 102.4 mm to (133.2, 138.5)
- moved R23 102.4 mm to (109.5, 73.8)
- moved R29 102.4 mm to (123.0, 105.0)
- moved D17 102.4 mm to (80.8, 88.1)
- moved D18 102.4 mm to (79.2, 73.8)
- moved D19 102.4 mm to (113.5, 73.8)
- moved D20 102.4 mm to (121.8, 120.1)
- moved D21 102.4 mm to (72.8, 120.1)
- moved D23 102.4 mm to (91.8, 54.1)
- moved D6 102.4 mm to (113.8, 88.1)
- moved D7 102.4 mm to (65.8, 104.7)
- moved D8 102.4 mm to (101.8, 54.1)
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Routing:
- net (no net): vias 0 -> 2
Other:
- outline, holes or cut-outs redrawn
- board text added: "JLCJLCJLCJLC"

Commit message: dodano gerbery bez napisu JLCJLCJLC
Other:
- board text removed: "JLCJLCJLCJLC"
